Commit message: use the default urdf from the open source project

File: config/anymal/model.urdf (robot description, URDF)
Before this commit: robot anymal, 36 links, 35 joints
Links:
- removed link dual_realsense_mount
- removed link dual_realsense_mount_tilted
- removed link handle_mount_front
- removed link handle_mount_front_sensor_mount_axis_aligned
- removed link imu_link
- removed link realsense_d435_front_camera
- removed link realsense_d435_front_camera_axis_aligned
- removed link realsense_d435_front_camera_parent
- removed link realsense_d435_front_forward_camera
- removed link realsense_d435_front_forward_camera_axis_aligned
- removed link realsense_d435_front_forward_camera_parent
- removed link velodyne
- removed link velodyne_axis_aligned
- removed link velodyne_mount
- link LF_ADAPTER: geometry collision cylinder length=0.32125 radius=0.015; visual mesh filename=package://anymal_b_simple_description/meshes/anymal_foot.dae scale=0.001 0.001 0.001
- link LF_THIGH: geometry collision box size=0.08 0.04 0.25; collision cylinder length=0.12 radius=0.06
- link LH_ADAPTER: geometry collision cylinder length=0.32125 radius=0.015; visual mesh filename=package://anymal_b_simple_description/meshes/anymal_foot.dae scale=0.001 0.001 0.001
- link LH_THIGH: geometry collision box size=0.08 0.04 0.25; collision cylinder length=0.12 radius=0.06
- link RF_ADAPTER: geometry collision cylinder length=0.32125 radius=0.015; visual mesh filename=package://anymal_b_simple_description/meshes/anymal_foot.dae scale=0.001 0.001 0.001
- link RF_THIGH: geometry collision box size=0.08 0.04 0.25; collision cylinder length=0.12 radius=0.06
- link RH_ADAPTER: geometry collision cylinder length=0.32125 radius=0.015; visual mesh filename=package://anymal_b_simple_description/meshes/anymal_foot.dae scale=0.001 0.001 0.001
- link RH_THIGH: geometry collision box size=0.08 0.04 0.25; collision cylinder length=0.12 radius=0.06
Joints:
- removed joint base_to_handle_mount_front_axis_aligned
- removed joint base_to_velodyne_mount
- removed joint dual_realsense_mount_tilted_to_realsense_d435_front_camera_axis_aligned
- removed joint dual_realsense_mount_tilted_to_realsense_d435_front_forward_camera_axis_aligned
- removed joint dual_realsense_mount_to_dual_realsense_mount_tilted
- removed joint handle_mount_front_sensor_mount_axis_aligned_to_dual_realsense_mount
- removed joint handle_mount_front_to_sensor_mount_axis_aligned
- removed joint imu_joint
- removed joint realsense_d435_front_camera_axis_aligned_to_camera
- removed joint realsense_d435_front_camera_to_camera_parent
- removed joint realsense_d435_front_forward_camera_axis_aligned_to_camera
- removed joint realsense_d435_front_forward_camera_to_camera_parent
- removed joint velodyne_axis_aligned_to_velodyne
- removed joint velodyne_mount_to_velodyne_axis_aligned
